File: kicad/FroyOutdoor/FroyOutdoor.sch (KiCad schematic (older format))
At the start: 23 parts, among them IC1 ESP-WROOM-02U__4MB_, J1 Conn_01x06, Q1 Q_NPN_BEC, Q2 Q_NPN_BEC, Q3 Q_NPN_BEC, SW1 SW_SPST, U2 BME280

Commit message: Froy Outdoor 2.1, now with transistor controlling sensor and battery measurement
Parts:
- added Q4: Q_NPN_BEC, Package_TO_SOT_SMD:SOT-23, symbol Device:Q_NPN_BEC
- R4: renamed from R11; value 12k -> 10k
- R5: renamed from R9; value 12k -> 10k
- R6: renamed from R8; value 12k -> 10k
- renumbered R5 to R10, R4 to R11, R6 to R2, R2 to R7, R7 to R8, R10 to R9
Connections:
- net +3V3: now also Q4.3 (C); no longer C2.2, R1.1, R2.1, R8.1, U2.2 (CSB), U2.6 (VDDIO), U2.8 (VDD)
- net PWR_ENABLE: now reaches IC1.4 (IO12)
- net PWR_ENABLE: now also Q4.1 (B)
- new net +3.3VP: C2.2, Q4.2 (E), R1.1, R2.1, R8.1, U2.2 (CSB), U2.6 (VDDIO), U2.8 (VDD)
- no-connect marks 3 -> 2
Other:
- note added: "Power for sensor/battery measurement"
Changed lines of the file:
@@
 RST
 $Comp
-L Device:R R9
+L Device:R R5
 U 1 1 608F39ED
 P 5700 6400
-F 0 "R9" V 5493 6400 50  0000 C CNN
-F 1 "12k" V 5584 6400 50  0000 C CNN
+F 0 "R5" V 5493 6400 50  0000 C CNN
+F 1 "10k" V 5584 6400 50  0000 C CNN
 F 2 "Resistor_SMD:R_0805_2012Metric" V 5630 6400 50  0001 C CNN
 F 3 "~" H 5700 6400 50  0001 C CNN
@@
 	6900 7150 6900 7250
 $Comp
-L Device:R R4
+L Device:R R11
 U 1 1 607C09B0
 P 4650 3700
-F 0 "R4" H 4580 3654 50  0000 R CNN
+F 0 "R11" H 4580 3654 50  0000 R CNN
 F 1 "10k" H 4580 3745 50  0000 R CNN
 F 2 "Resistor_SMD:R_0805_2012Metric" V 4580 3700 50  0001 C CNN
@@
 $EndComp
 $Comp
-L Device:R R2
+L Device:R R7
 U 1 1 607A274F
 P 3200 2350
-F 0 "R2" H 3130 2396 50  0000 R CNN
+F 0 "R7" H 3130 2396 50  0000 R CNN
 F 1 "10k" H 3130 2305 50  0000 R CNN
 F 2 "Resistor_SMD:R_0805_2012Metric" V 3130 2350 50  0001 C CNN
@@
 Text Notes 3050 1250 0    100  ~ 0
 ESP-WROOM-02U/D
-Text Label 5300 3250 2    50   ~ 0
+Text Label 5400 3250 2    50   ~ 0
 I2C_CLK
-Text Label 5300 2750 2    50   ~ 0
+Text Label 5400 2750 2    50   ~ 0
 I2C_SDA
-Text Label 5300 2650 2    50   ~ 0
+Text Label 5400 2650 2    50   ~ 0
 IO0
 Text Label 2550 2800 0    50   ~ 0
@@
 TXD
 Wire Wire Line
-	4600 2750 5300 2750
-Wire Wire Line
-	4600 3250 5300 3250
+	4600 2750 5400 2750
+Wire Wire Line
+	4600 3250 5400 3250
 Wire Wire Line
 	3400 2700 3200 2700
@@
 $EndComp
 Wire Wire Line
-	4600 2650 5300 2650
-NoConn ~ 4600 3050
+	4600 2650 5400 2650
 NoConn ~ 4600 3150
 NoConn ~ 4600 2850
@@
 $EndComp
 $Comp
-L Device:R R5
+L Device:R R10
 U 1 1 607C9920
 P 3250 5750
-F 0 "R5" V 3043 5750 50  0000 C CNN
+F 0 "R10" V 3043 5750 50  0000 C CNN
 F 1 "2k2" V 3134 5750 50  0000 C CNN
 F 2 "Resistor_SMD:R_0805_2012Metric" V 3180 5750 50  0001 C CNN
@@
 $EndComp
 Wire Wire Line
-	4600 2950 5300 2950
-Text Label 5300 2950 2    50   ~ 0
+	4600 2950 5400 2950
+Text Label 5400 2950 2    50   ~ 0
 LED
 $Comp
-L Device:R R8
+L Device:R R6
 U 1 1 6086724D
 P 5700 7000
-F 0 "R8" V 5815 7000 50  0000 C CNN
-F 1 "12k" V 5906 7000 50  0000 C CNN
+F 0 "R6" V 5815 7000 50  0000 C CNN
+F 1 "10k" V 5906 7000 50  0000 C CNN
 F 2 "Resistor_SMD:R_0805_2012Metric" V 5630 7000 50  0001 C CNN
 F 3 "~" H 5700 7000 50  0001 C CNN
@@
 BME280/680
 $Comp
-L power:+3V3 #PWR0103
-U 1 1 60A86F8A
-P 6550 2150
-F 0 "#PWR0103" H 6550 2000 50  0001 C CNN
-F 1 "+3V3" H 6565 2323 50  0000 C CNN
-F 2 "" H 6550 2150 50  0001 C CNN
-F 3 "" H 6550 2150 50  0001 C CNN
-	1    6550 2150
-	1    0    0    -1
-$EndComp
-$Comp
 L power:+3V3 #PWR0106
 U 1 1 60A8BC25
@@
 $EndComp
 Wire Wire Line
-	4600 3450 5300 3450
-Text Label 5300 3450 2    50   ~ 0
+	4600 3450 5400 3450
+Text Label 5400 3450 2    50   ~ 0
 WAKE_UP
 Text Label 4800 5600 0    50   ~ 0
@@
 Connection ~ 5300 6650
 $Comp
-L Device:R R11
+L Device:R R4
 U 1 1 60BF9F09
 P 5700 5900
-F 0 "R11" V 5493 5900 50  0000 C CNN
-F 1 "12k" V 5584 5900 50  0000 C CNN
+F 0 "R4" V 5493 5900 50  0000 C CNN
+F 1 "10k" V 5584 5900 50  0000 C CNN
 F 2 "Resistor_SMD:R_0805_2012Metric" V 5630 5900 50  0001 C CNN
 F 3 "~" H 5700 5900 50  0001 C CNN
@@
 	8550 6550 8550 6650
 $Comp
-L Device:R R6
+L Device:R R2
 U 1 1 60D714B3
 P 8850 6400
-F 0 "R6" H 8780 6446 50  0000 R CNN
+F 0 "R2" H 8780 6446 50  0000 R CNN
 F 1 "4k7" H 8780 6355 50  0000 R CNN
 F 2 "Resistor_SMD:R_0805_2012Metric" V 8780 6400 50  0001 C CNN
@@
 Wire Wire Line
 	7900 6850 8850 6850
-$Comp
-L power:+3V3 #PWR06
-U 1 1 60D73F62
-P 8700 6000
-F 0 "#PWR06" H 8700 5850 50  0001 C CNN
-F 1 "+3V3" H 8715 6173 50  0000 C CNN
-F 2 "" H 8700 6000 50  0001 C CNN
-F 3 "" H 8700 6000 50  0001 C CNN
-	1    8700 6000
-	1    0    0    -1
-$EndComp
 Wire Wire Line
 	8700 6100 8550 6100
@@
 BATT_SENS
 $Comp
-L Device:R R7
+L Device:R R8
 U 1 1 60E62BD0
 P 1450 6100
-F 0 "R7" H 1380 6146 50  0000 R CNN
+F 0 "R8" H 1380 6146 50  0000 R CNN
 F 1 "47k" H 1380 6055 50  0000 R CNN
 F 2 "Resistor_SMD:R_0805_2012Metric" V 1380 6100 50  0001 C CNN
@@
 $EndComp
 $Comp
-L Device:R R10
+L Device:R R9
 U 1 1 60E6326F
 P 1450 6600
-F 0 "R10" H 1380 6646 50  0000 R CNN
+F 0 "R9" H 1380 6646 50  0000 R CNN
 F 1 "22k" H 1380 6555 50  0000 R CNN
 F 2 "Resistor_SMD:R_0805_2012Metric" V 1380 6600 50  0001 C CNN
@@
 	1    1450 6600
 	-1   0    0    -1
-$EndComp
-$Comp
-L power:+3V3 #PWR08
-U 1 1 60E636CB
-P 1450 5800
-F 0 "#PWR08" H 1450 5650 50  0001 C CNN
-F 1 "+3V3" H 1465 5973 50  0000 C CNN
-F 2 "" H 1450 5800 50  0001 C CNN
-F 3 "" H 1450 5800 50  0001 C CNN
-	1    1450 5800
-	1    0    0    -1
 $EndComp
 Wire Wire Line
@@
 Wire Wire Line
 	4000 1600 4000 2100
+$Comp
+L Device:Q_NPN_BEC Q4
+U 1 1 61409855
+P 6250 8650
+F 0 "Q4" H 6441 8696 50  0000 L CNN
+F 1 "Q_NPN_BEC" H 6441 8605 50  0000 L CNN
+F 2 "Package_TO_SOT_SMD:SOT-23" H 6450 8750 50  0001 C CNN
+F 3 "~" H 6250 8650 50  0001 C CNN
+	1    6250 8650
+	1    0    0    -1
+$EndComp
+$Comp
+L power:+3V3 #PWR0102
+U 1 1 6140A42A
+P 6350 8250
+F 0 "#PWR0102" H 6350 8100 50  0001 C CNN
+F 1 "+3V3" H 6365 8423 50  0000 C CNN
+F 2 "" H 6350 8250 50  0001 C CNN
+F 3 "" H 6350 8250 50  0001 C CNN
+	1    6350 8250
+	1    0    0    -1
+$EndComp
+Wire Wire Line
+	6350 8450 6350 8250
+$Comp
+L power:+3.3VP #PWR0103
+U 1 1 6140EF27
+P 6350 9050
+F 0 "#PWR0103" H 6500 9000 50  0001 C CNN
+F 1 "+3.3VP" H 6365 9223 50  0000 C CNN
+F 2 "" H 6350 9050 50  0001 C CNN
+F 3 "" H 6350 9050 50  0001 C CNN
+	1    6350 9050
+	-1   0    0    1
+$EndComp
+Wire Wire Line
+	6350 8850 6350 9050
+Text Label 5400 8650 0    50   ~ 0
+PWR_ENABLE
+Wire Wire Line
+	6050 8650 5400 8650
+Wire Notes Line
+	6950 9350 6950 7950
+Wire Notes Line
+	6950 7950 5950 7950
+Wire Notes Line
+	5950 7950 5950 9350
+Wire Notes Line
+	5950 9350 6950 9350
+Text Notes 5950 7900 0    50   ~ 0
+Power for sensor/battery measurement
+$Comp
+L power:+3.3VP #PWR0104
+U 1 1 6142BD0F
+P 8700 6000
+F 0 "#PWR0104" H 8850 5950 50  0001 C CNN
+F 1 "+3.3VP" H 8715 6173 50  0000 C CNN
+F 2 "" H 8700 6000 50  0001 C CNN
+F 3 "" H 8700 6000 50  0001 C CNN
+	1    8700 6000
+	1    0    0    -1
+$EndComp
+$Comp
+L power:+3.3VP #PWR0105
+U 1 1 6142E1CD
+P 6550 2150
+F 0 "#PWR0105" H 6700 2100 50  0001 C CNN
+F 1 "+3.3VP" H 6565 2323 50  0000 C CNN
+F 2 "" H 6550 2150 50  0001 C CNN
+F 3 "" H 6550 2150 50  0001 C CNN
+	1    6550 2150
+	1    0    0    -1
+$EndComp
+Text Label 5400 3050 2    50   ~ 0
+PWR_ENABLE
+Wire Wire Line
+	4600 3050 5400 3050
+$Comp
+L power:+3.3VP #PWR0107
+U 1 1 61452289
+P 1450 5800
+F 0 "#PWR0107" H 1600 5750 50  0001 C CNN
+F 1 "+3.3VP" H 1465 5973 50  0000 C CNN
+F 2 "" H 1450 5800 50  0001 C CNN
+F 3 "" H 1450 5800 50  0001 C CNN
+	1    1450 5800
+	1    0    0    -1
+$EndComp
 $EndSCHEMATC

Commit message: FroyOutdoor v2.2 - removed power transistor again, used Omron button
Parts:
- removed Q4: Q_NPN_BEC, Package_TO_SOT_SMD:SOT-23, symbol Device:Q_NPN_BEC
- removed SW1: SW_SPST, Button_Switch_SMD:SW_SPST_CK_RS282G05A3, symbol Switch:SW_SPST
- added SW1: SW_MEC_5E, xrstf:SW_SPST_Omron_B3FS-100xP, symbol Switch:SW_MEC_5E
- D1: footprint LED_SMD:LED_1206_3216Metric_Pad1.42x1.75mm_HandSolder -> LED_SMD:LED_0805_2012Metric
- R1, R2: value 4k7 -> 10k
- R8: value 47k -> 4M7
- R9: value 22k -> 2M2
Connections:
- net +3.3VP is gone; now on net +3V3: C2.2, R1.1, R2.1, R8.1, U2.2 (CSB), U2.6 (VDDIO), U2.8 (VDD)
- net GNDREF: now also SW1.3 (K)
- net RST: now also SW1.1
- net PWR_ENABLE: no longer names the net of IC1.4 (IO12)
- no-connect marks 2 -> 5
Other:
- note added: "(4 pins because the 2-pin SPST\nbutton is not available at reichelt)"
- note removed: "Power for sensor/battery measurement"
Changed lines of the file:
@@
 F 0 "D1" H 3643 5967 50  0000 C CNN
 F 1 "STATUS" H 3643 5876 50  0000 C CNN
-F 2 "LED_SMD:LED_1206_3216Metric_Pad1.42x1.75mm_HandSolder" H 3650 5750 50  0001 C CNN
+F 2 "LED_SMD:LED_0805_2012Metric" H 3650 5750 50  0001 C CNN
 F 3 "~" H 3650 5750 50  0001 C CNN
 	1    3650 5750
@@
 Wire Wire Line
 	4050 5750 4050 5900
-$Comp
-L Switch:SW_SPST SW1
-U 1 1 60A341F2
-P 3500 6950
-F 0 "SW1" H 3500 7185 50  0000 C CNN
-F 1 "SW_SPST" H 3500 7094 50  0000 C CNN
-F 2 "Button_Switch_SMD:SW_SPST_CK_RS282G05A3" H 3500 6950 50  0001 C CNN
-F 3 "~" H 3500 6950 50  0001 C CNN
-	1    3500 6950
-	1    0    0    -1
-$EndComp
-Wire Wire Line
-	3300 6950 2900 6950
 Text Label 2900 6950 0    50   ~ 0
 RST
@@
 	1    0    0    -1
 $EndComp
-Wire Wire Line
-	3700 6950 3800 6950
-Wire Wire Line
-	3800 6950 3800 7150
 Wire Notes Line
 	3150 7450 4050 7450
@@
 P 8550 6400
 F 0 "R1" H 8480 6446 50  0000 R CNN
-F 1 "4k7" H 8480 6355 50  0000 R CNN
+F 1 "10k" H 8480 6355 50  0000 R CNN
 F 2 "Resistor_SMD:R_0805_2012Metric" V 8480 6400 50  0001 C CNN
 F 3 "~" H 8550 6400 50  0001 C CNN
@@
 P 8850 6400
 F 0 "R2" H 8780 6446 50  0000 R CNN
-F 1 "4k7" H 8780 6355 50  0000 R CNN
+F 1 "10k" H 8780 6355 50  0000 R CNN
 F 2 "Resistor_SMD:R_0805_2012Metric" V 8780 6400 50  0001 C CNN
 F 3 "~" H 8850 6400 50  0001 C CNN
@@
 P 1450 6100
 F 0 "R8" H 1380 6146 50  0000 R CNN
-F 1 "47k" H 1380 6055 50  0000 R CNN
+F 1 "4M7" H 1380 6055 50  0000 R CNN
 F 2 "Resistor_SMD:R_0805_2012Metric" V 1380 6100 50  0001 C CNN
 F 3 "~" H 1450 6100 50  0001 C CNN
 	1    1450 6100
-	-1   0    0    -1
-$EndComp
-$Comp
-L Device:R R9
-U 1 1 60E6326F
-P 1450 6600
-F 0 "R9" H 1380 6646 50  0000 R CNN
-F 1 "22k" H 1380 6555 50  0000 R CNN
-F 2 "Resistor_SMD:R_0805_2012Metric" V 1380 6600 50  0001 C CNN
-F 3 "~" H 1450 6600 50  0001 C CNN
-	1    1450 6600
 	-1   0    0    -1
 $EndComp
@@
 	4000 1600 4000 2100
 $Comp
-L Device:Q_NPN_BEC Q4
-U 1 1 61409855
-P 6250 8650
-F 0 "Q4" H 6441 8696 50  0000 L CNN
-F 1 "Q_NPN_BEC" H 6441 8605 50  0000 L CNN
-F 2 "Package_TO_SOT_SMD:SOT-23" H 6450 8750 50  0001 C CNN
-F 3 "~" H 6250 8650 50  0001 C CNN
-	1    6250 8650
-	1    0    0    -1
-$EndComp
-$Comp
 L power:+3V3 #PWR0102
-U 1 1 6140A42A
-P 6350 8250
-F 0 "#PWR0102" H 6350 8100 50  0001 C CNN
-F 1 "+3V3" H 6365 8423 50  0000 C CNN
-F 2 "" H 6350 8250 50  0001 C CNN
-F 3 "" H 6350 8250 50  0001 C CNN
-	1    6350 8250
-	1    0    0    -1
-$EndComp
-Wire Wire Line
-	6350 8450 6350 8250
-$Comp
-L power:+3.3VP #PWR0103
-U 1 1 6140EF27
-P 6350 9050
-F 0 "#PWR0103" H 6500 9000 50  0001 C CNN
-F 1 "+3.3VP" H 6365 9223 50  0000 C CNN
-F 2 "" H 6350 9050 50  0001 C CNN
-F 3 "" H 6350 9050 50  0001 C CNN
-	1    6350 9050
-	-1   0    0    1
-$EndComp
-Wire Wire Line
-	6350 8850 6350 9050
-Text Label 5400 8650 0    50   ~ 0
-PWR_ENABLE
-Wire Wire Line
-	6050 8650 5400 8650
-Wire Notes Line
-	6950 9350 6950 7950
-Wire Notes Line
-	6950 7950 5950 7950
-Wire Notes Line
-	5950 7950 5950 9350
-Wire Notes Line
-	5950 9350 6950 9350
-Text Notes 5950 7900 0    50   ~ 0
-Power for sensor/battery measurement
-$Comp
-L power:+3.3VP #PWR0104
-U 1 1 6142BD0F
+U 1 1 614B5C05
 P 8700 6000
-F 0 "#PWR0104" H 8850 5950 50  0001 C CNN
-F 1 "+3.3VP" H 8715 6173 50  0000 C CNN
+F 0 "#PWR0102" H 8700 5850 50  0001 C CNN
+F 1 "+3V3" H 8715 6173 50  0000 C CNN
 F 2 "" H 8700 6000 50  0001 C CNN
 F 3 "" H 8700 6000 50  0001 C CNN
@@
 $EndComp
 $Comp
-L power:+3.3VP #PWR0105
-U 1 1 6142E1CD
+L power:+3V3 #PWR0103
+U 1 1 614B7A85
 P 6550 2150
-F 0 "#PWR0105" H 6700 2100 50  0001 C CNN
-F 1 "+3.3VP" H 6565 2323 50  0000 C CNN
+F 0 "#PWR0103" H 6550 2000 50  0001 C CNN
+F 1 "+3V3" H 6565 2323 50  0000 C CNN
 F 2 "" H 6550 2150 50  0001 C CNN
 F 3 "" H 6550 2150 50  0001 C CNN
@@
 	1    0    0    -1
 $EndComp
-Text Label 5400 3050 2    50   ~ 0
-PWR_ENABLE
-Wire Wire Line
-	4600 3050 5400 3050
-$Comp
-L power:+3.3VP #PWR0107
-U 1 1 61452289
+$Comp
+L power:+3V3 #PWR0104
+U 1 1 614BB4BA
 P 1450 5800
-F 0 "#PWR0107" H 1600 5750 50  0001 C CNN
-F 1 "+3.3VP" H 1465 5973 50  0000 C CNN
+F 0 "#PWR0104" H 1450 5650 50  0001 C CNN
+F 1 "+3V3" H 1465 5973 50  0000 C CNN
 F 2 "" H 1450 5800 50  0001 C CNN
 F 3 "" H 1450 5800 50  0001 C CNN
@@
 	1    0    0    -1
 $EndComp
+$Comp
+L Device:R R9
+U 1 1 60E6326F
+P 1450 6600
+F 0 "R9" H 1380 6646 50  0000 R CNN
+F 1 "2M2" H 1380 6555 50  0000 R CNN
+F 2 "Resistor_SMD:R_0805_2012Metric" V 1380 6600 50  0001 C CNN
+F 3 "~" H 1450 6600 50  0001 C CNN
+	1    1450 6600
+	-1   0    0    -1
+$EndComp
+NoConn ~ 4600 3050
+$Comp
+L Switch:SW_MEC_5E SW1
+U 1 1 6151A03B
+P 3500 7050
+F 0 "SW1" H 3500 7435 50  0000 C CNN
+F 1 "SW_MEC_5E" H 3500 7344 50  0000 C CNN
+F 2 "xrstf:SW_SPST_Omron_B3FS-100xP" H 3500 7350 50  0001 C CNN
+F 3 "http://www.apem.com/int/index.php?controller=attachment&id_attachment=1371" H 3500 7350 50  0001 C CNN
+	1    3500 7050
+	1    0    0    -1
+$EndComp
+Wire Wire Line
+	3700 7050 3800 7050
+Wire Wire Line
+	3800 7050 3800 7150
+Text Notes 2950 7650 0    50   ~ 0
+(4 pins because the 2-pin SPST\nbutton is not available at reichelt)
+Wire Wire Line
+	2900 6950 3300 6950
+NoConn ~ 3700 6950
+NoConn ~ 3300 7050
 $EndSCHEMATC

Commit message: FroyOutdoor v2.3 - expose I2C SDA/SCL pins to make it easy to reuse the board for quick experiments with other breakout boards
Parts:
- J1: value Conn_01x06 -> Conn_01x08; footprint xrstf:PinHeader_1x06_P2.54mm_Vertical -> xrstf:PinHeader_1x08_P2.54mm_Vertical; symbol Connector_Generic:Conn_01x06 -> Connector_Generic:Conn_01x08
Connections:
- net +3V3: now also J1.3 (Pin_3); no longer J1.1 (Pin_1)
- net DTR: now also J1.7 (Pin_7); no longer J1.5 (Pin_5)
- net GNDREF: now also J1.4 (Pin_4); no longer J1.2 (Pin_2)
- net I2C_CLK: now also J1.1 (Pin_1)
- net I2C_SDA: now also J1.2 (Pin_2)
- net RTS: now also J1.8 (Pin_8); no longer J1.6 (Pin_6)
- net RXD: now also J1.6 (Pin_6); no longer J1.4 (Pin_4)
- net TXD: now also J1.5 (Pin_5); no longer J1.3 (Pin_3)
Changed lines of the file:
@@
 I²C Pull Ups
 $Comp
-L Connector_Generic:Conn_01x06 J1
+L Connector_Generic:Conn_01x08 J1
 U 1 1 60DD9688
 P 1150 4100
 F 0 "J1" H 1068 3575 50  0000 C CNN
-F 1 "Conn_01x06" H 1068 3666 50  0000 C CNN
-F 2 "xrstf:PinHeader_1x06_P2.54mm_Vertical" H 1150 4100 50  0001 C CNN
+F 1 "Conn_01x08" H 1068 3666 50  0000 C CNN
+F 2 "xrstf:PinHeader_1x08_P2.54mm_Vertical" H 1150 4100 50  0001 C CNN
 F 3 "~" H 1150 4100 50  0001 C CNN
 	1    1150 4100
@@
 L power:+3V3 #PWR03
 U 1 1 60DE945E
-P 1550 3600
-F 0 "#PWR03" H 1550 3450 50  0001 C CNN
-F 1 "+3V3" H 1565 3773 50  0000 C CNN
-F 2 "" H 1550 3600 50  0001 C CNN
-F 3 "" H 1550 3600 50  0001 C CNN
-	1    1550 3600
+P 1550 3500
+F 0 "#PWR03" H 1550 3350 50  0001 C CNN
+F 1 "+3V3" H 1565 3673 50  0000 C CNN
+F 2 "" H 1550 3500 50  0001 C CNN
+F 3 "" H 1550 3500 50  0001 C CNN
+	1    1550 3500
 	1    0    0    -1
 $EndComp
@@
 L power:GNDREF #PWR05
 U 1 1 60DE9B71
-P 1650 4450
-F 0 "#PWR05" H 1650 4200 50  0001 C CNN
-F 1 "GNDREF" H 1655 4277 50  0000 C CNN
-F 2 "" H 1650 4450 50  0001 C CNN
-F 3 "" H 1650 4450 50  0001 C CNN
-	1    1650 4450
-	-1   0    0    -1
-$EndComp
-Wire Wire Line
-	1350 4300 1550 4300
-Wire Wire Line
-	1550 4300 1550 3600
-Wire Wire Line
-	1350 4200 1650 4200
-Wire Wire Line
-	1650 4200 1650 4450
-Wire Wire Line
-	1350 4100 2150 4100
-Text Label 2150 4100 2    50   ~ 0
+P 1650 4550
+F 0 "#PWR05" H 1650 4300 50  0001 C CNN
+F 1 "GNDREF" H 1655 4377 50  0000 C CNN
+F 2 "" H 1650 4550 50  0001 C CNN
+F 3 "" H 1650 4550 50  0001 C CNN
+	1    1650 4550
+	-1   0    0    -1
+$EndComp
+Wire Wire Line
+	1350 4200 1550 4200
+Wire Wire Line
+	1550 4200 1550 3500
+Wire Wire Line
+	1350 4100 1650 4100
+Wire Wire Line
+	1650 4100 1650 4550
+Wire Wire Line
+	1350 4000 2250 4000
+Text Label 2250 4000 2    50   ~ 0
 TXD
 Wire Wire Line
-	1350 4000 2150 4000
-Wire Wire Line
-	1350 3900 2150 3900
-Wire Wire Line
-	1350 3800 2150 3800
-Text Label 2150 4000 2    50   ~ 0
+	1350 3900 2250 3900
+Wire Wire Line
+	1350 3800 2250 3800
+Wire Wire Line
+	1350 3700 2250 3700
+Text Label 2250 3900 2    50   ~ 0
 RXD
-Text Label 2150 3900 2    50   ~ 0
+Text Label 2250 3800 2    50   ~ 0
 DTR
-Text Label 2150 3800 2    50   ~ 0
+Text Label 2250 3700 2    50   ~ 0
 RTS
 Wire Notes Line
-	1900 4750 1900 3300
-Wire Notes Line
-	1900 3300 900  3300
-Wire Notes Line
-	900  3300 900  4750
-Wire Notes Line
-	900  4750 1900 4750
-Text Notes 900  3250 0    100  ~ 0
+	1900 4850 1900 3200
+Wire Notes Line
+	1900 3200 900  3200
+Wire Notes Line
+	900  3200 900  4850
+Wire Notes Line
+	900  4850 1900 4850
+Text Notes 900  3150 0    100  ~ 0
 Progr. Port
 Wire Wire Line
@@
 NoConn ~ 3700 6950
 NoConn ~ 3300 7050
+Wire Wire Line
+	1350 4300 2250 4300
+Wire Wire Line
+	1350 4400 2250 4400
+Text Label 2250 4300 2    50   ~ 0
+I2C_SDA
+Text Label 2250 4400 2    50   ~ 0
+I2C_CLK
 $EndSCHEMATC
