File: kicad/FroyIndoor/FroyIndoor.kicad_pcb (KiCad board)
At the start: 2 copper layers, 80 x 60 mm, 37 parts, among them IC1 ESP-WROOM-02U__4MB_, J1 USB_B_Mini, J2 BME260_Breakout, Q1 Q_NPN_BEC, Q2 Q_NPN_BEC, Q3 Q_NPN_BEC, SW1 SW_SPST, U1 FT232RL, U2 BME280

Commit message: FroyIndoor v1.2.1 - fix silk screen for the I2C pins, use more common resistor values
Other:
- board text added: "10k 10k 10k 10k 2k2 2k2 2k2 10k 10k 10k 10k 10k 10k"
- board text added: "2021-10-10"
- board text added: "Frøy Indoor 1.2.1"
- board text removed: "10k 10k 10k 10k 270 270 270 12k 12k 10k 12k 10k 10k"
- board text removed: "2021-06-25"
- board text removed: "Arduino IDE settings: -> Generic ESP8266 Board -> Reset mode: dtr (aka nodemcu) -> Flash Size: 2MB (FS: 64KB) -> Flash Frequency: 26MHz"
- board text removed: "Frøy Indoor 1.2"
- board text removed: "I²C:"
- board text removed: "SDA on GPIO2 SCK on GPIO14 This is not the default for ESP8266 boards in Arduino!"
