File: kicad/FroyIndoor/FroyIndoor.sch (KiCad schematic (older format))
At the start: 32 parts, among them IC1 ESP-WROOM-02U__4MB_, J1 USB_B_Mini, J2 BME260_Breakout, Q1 Q_NPN_BEC, Q2 Q_NPN_BEC, Q3 Q_NPN_BEC, SW1 SW_SPST, U1 FT232RL, U2 BME280

Commit message: FroyIndoor v1.2.1 - fix silk screen for the I2C pins, use more common resistor values
Parts:
- R11, R8, R9: value 12k -> 10k
- R5, R6, R7: value 270 -> 2k2
Changed lines of the file:
@@
 P 6150 6300
 F 0 "R9" V 5943 6300 50  0000 C CNN
-F 1 "12k" V 6034 6300 50  0000 C CNN
+F 1 "10k" V 6034 6300 50  0000 C CNN
 F 2 "Resistor_SMD:R_1206_3216Metric_Pad1.42x1.75mm_HandSolder" V 6080 6300 50  0001 C CNN
 F 3 "~" H 6150 6300 50  0001 C CNN
@@
 P 3300 6350
 F 0 "R6" V 3093 6350 50  0000 C CNN
-F 1 "270" V 3184 6350 50  0000 C CNN
+F 1 "2k2" V 3184 6350 50  0000 C CNN
 F 2 "Resistor_SMD:R_1206_3216Metric_Pad1.42x1.75mm_HandSolder" V 3230 6350 50  0001 C CNN
 F 3 "~" H 3300 6350 50  0001 C CNN
@@
 P 3300 6750
 F 0 "R7" V 3093 6750 50  0000 C CNN
-F 1 "270" V 3184 6750 50  0000 C CNN
+F 1 "2k2" V 3184 6750 50  0000 C CNN
 F 2 "Resistor_SMD:R_1206_3216Metric_Pad1.42x1.75mm_HandSolder" V 3230 6750 50  0001 C CNN
 F 3 "~" H 3300 6750 50  0001 C CNN
@@
 P 3300 5950
 F 0 "R5" V 3093 5950 50  0000 C CNN
-F 1 "270" V 3184 5950 50  0000 C CNN
+F 1 "2k2" V 3184 5950 50  0000 C CNN
 F 2 "Resistor_SMD:R_1206_3216Metric_Pad1.42x1.75mm_HandSolder" V 3230 5950 50  0001 C CNN
 F 3 "~" H 3300 5950 50  0001 C CNN
@@
 P 6150 6900
 F 0 "R8" V 6265 6900 50  0000 C CNN
-F 1 "12k" V 6356 6900 50  0000 C CNN
+F 1 "10k" V 6356 6900 50  0000 C CNN
 F 2 "Resistor_SMD:R_1206_3216Metric_Pad1.42x1.75mm_HandSolder" V 6080 6900 50  0001 C CNN
 F 3 "~" H 6150 6900 50  0001 C CNN
@@
 P 6150 5800
 F 0 "R11" V 5943 5800 50  0000 C CNN
-F 1 "12k" V 6034 5800 50  0000 C CNN
+F 1 "10k" V 6034 5800 50  0000 C CNN
 F 2 "Resistor_SMD:R_1206_3216Metric_Pad1.42x1.75mm_HandSolder" V 6080 5800 50  0001 C CNN
 F 3 "~" H 6150 5800 50  0001 C CNN
