File: kicad/FroyLogger/FroyLogger.sch (KiCad schematic (older format))
At the start: 29 parts, among them J1 Conn_01x08, J2 Conn_01x04, J3 Conn_01x06, Q1 Q_NPN_BEC, Q2 Q_NPN_BEC, Q3 Q_NPN_BEC, SW1 SW_MEC_5E, U1 ESP-WROOM-02U__4MB_, U2 BME280, U3 MCP7940N-xSN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

Commit message: FroyLogger 3.0.1, better crystal footprint
Parts:
- Y1: footprint Crystal:Crystal_SMD_SeikoEpson_MC306-4Pin_8.0x3.2mm -> Crystal:Crystal_SMD_SeikoEpson_MC405-2Pin_9.6x4.1mm
Changed lines of the file:
@@
 F 0 "Y1" V 10004 3031 50  0000 L CNN
 F 1 "Crystal" V 10095 3031 50  0000 L CNN
-F 2 "Crystal:Crystal_SMD_SeikoEpson_MC306-4Pin_8.0x3.2mm" H 10050 2900 50  0001 C CNN
+F 2 "Crystal:Crystal_SMD_SeikoEpson_MC405-2Pin_9.6x4.1mm" H 10050 2900 50  0001 C CNN
 F 3 "~" H 10050 2900 50  0001 C CNN
 	1    10050 2900
